Commit message: Convert the single robotic arm to a dual-arm system, and adjust the simulation scene (remove the outer wall).

File: src/ur5e_gripper_moveit_config/urdf/ur5e_gripper.urdf.xacro (robot description, xacro)
@@ -4,6 +4,9 @@
     <link name="world"/>
     <xacro:include filename="single_ur5e_gripper.urdf.xacro" />
-    <xacro:ur5e_gripper name="ur" prefix="" parent="world" initial_positions_file="$(arg initial_positions_file)">
-        <origin xyz="0.3 0 1.03" rpy="0 0 0" />
+    <xacro:ur5e_gripper name="left_ur" prefix="" parent="world" initial_positions_file="$(arg initial_positions_file)">
+        <origin xyz="-0.275 0 1.03" rpy="0 0 0" />
+    </xacro:ur5e_gripper>
+    <xacro:ur5e_gripper name="right_ur" prefix="right_" parent="world" initial_positions_file="$(arg initial_positions_file)">
+        <origin xyz="1.075 0 1.03" rpy="0 0 3.1415926" />
     </xacro:ur5e_gripper>
     <xacro:arg name="use_nominal_extrinsics" default="true"/>
@@ -22,5 +25,5 @@
         <plugin name="gazebo_grasp_fix" filename="libgazebo_grasp_fix.so">
             <arm>
-                <arm_name>robotiq_gripper_arm</arm_name>
+                <arm_name>left_gripper_arm</arm_name>
                 <palm_link>wrist_3_link</palm_link>
                 <gripper_link>robotiq_85_left_finger_tip_link</gripper_link>
@@ -30,4 +33,14 @@
                 <gripper_link>robotiq_85_left_inner_knuckle_link</gripper_link>
                 <gripper_link>robotiq_85_right_inner_knuckle_link</gripper_link>
+            </arm>
+            <arm>
+                <arm_name>right_gripper_arm</arm_name>
+                <palm_link>right_wrist_3_link</palm_link>
+                <gripper_link>right_robotiq_85_left_finger_tip_link</gripper_link>
+                <gripper_link>right_robotiq_85_right_finger_tip_link</gripper_link>
+                <gripper_link>right_robotiq_85_left_knuckle_link</gripper_link>
+                <gripper_link>right_robotiq_85_right_knuckle_link</gripper_link>
+                <gripper_link>right_robotiq_85_left_inner_knuckle_link</gripper_link>
+                <gripper_link>right_robotiq_85_right_inner_knuckle_link</gripper_link>
             </arm>
             <forces_angle_tolerance>150</forces_angle_tolerance>

Commit message: Remove the vision and OctoMap components, and fix some related issues.

File: src/ur5e_gripper_moveit_config/urdf/ur5e_gripper.urdf.xacro (robot description, xacro)
@@ -12,11 +12,4 @@
         <origin xyz="0.65 0 1.016" rpy="0 0 3.1415926" />
     </xacro:ur5e_gripper>
-    <xacro:arg name="use_nominal_extrinsics" default="true"/>
-    <xacro:arg name="add_plug" default="false" />
-    <xacro:arg name="use_mesh" default="true" />
-    <xacro:include filename="$(find realsense2_description)/urdf/_d435.urdf.xacro" />
-    <xacro:sensor_d435 parent="world" use_nominal_extrinsics="$(arg use_nominal_extrinsics)" add_plug="$(arg add_plug)" use_mesh="$(arg use_mesh)">
-        <origin xyz="1.5 0 2" rpy="0 0.785398163 3.1415926"/>
-    </xacro:sensor_d435>
     <gazebo>
         <plugin filename="libgazebo_ros2_control.so" name="gazebo_ros2_control">
