Commit message: Modify the dual-arm controller and further refine the scene layout.

File: src/ur5e_gripper_moveit_config/srdf/ur5e_gripper.srdf.xacro (robot description, xacro)
@@ -3,6 +3,12 @@
     <xacro:include filename="$(find ur_moveit_config)/srdf/ur_macro.srdf.xacro" />
     <xacro:ur_srdf name="ur" prefix="" />
+    <xacro:ur_srdf name="ur" prefix="right_" />
     <xacro:include filename="$(find robotiq_moveit_config)/srdf/robotiq_macro.srdf.xacro" />
     <xacro:robotiq_srdf prefix="" />
+    <xacro:robotiq_srdf prefix="right_" />
+    <group name="dual_arms">
+        <group name="ur_manipulator" />
+        <group name="right_ur_manipulator" />
+    </group>
     <group_state name="ready" group="ur_manipulator">
         <joint name="elbow_joint" value="1.5707" />
@@ -13,6 +19,31 @@
         <joint name="wrist_3_joint" value="0" />
     </group_state>
+    <group_state name="right_ready" group="right_ur_manipulator">
+        <joint name="right_elbow_joint" value="1.5707" />
+        <joint name="right_shoulder_lift_joint" value="-1.5707" />
+        <joint name="right_shoulder_pan_joint" value="0" />
+        <joint name="right_wrist_1_joint" value="-1.5707" />
+        <joint name="right_wrist_2_joint" value="-1.5707" />
+        <joint name="right_wrist_3_joint" value="0" />
+    </group_state>
+    <group_state name="dual_ready" group="dual_arms">
+        <joint name="elbow_joint" value="1.5707" />
+        <joint name="shoulder_lift_joint" value="-1.5707" />
+        <joint name="shoulder_pan_joint" value="0" />
+        <joint name="wrist_1_joint" value="-1.5707" />
+        <joint name="wrist_2_joint" value="-1.5707" />
+        <joint name="wrist_3_joint" value="0" />
+        <joint name="right_elbow_joint" value="1.5707" />
+        <joint name="right_shoulder_lift_joint" value="-1.5707" />
+        <joint name="right_shoulder_pan_joint" value="0" />
+        <joint name="right_wrist_1_joint" value="-1.5707" />
+        <joint name="right_wrist_2_joint" value="-1.5707" />
+        <joint name="right_wrist_3_joint" value="0" />
+    </group_state>
     <disable_collisions link1="robotiq_85_base_link" link2="wrist_1_link" reason="Never"/>
     <disable_collisions link1="robotiq_85_base_link" link2="wrist_2_link" reason="Never"/>
     <disable_collisions link1="robotiq_85_base_link" link2="wrist_3_link" reason="Adjacent"/>
+    <disable_collisions link1="right_robotiq_85_base_link" link2="right_wrist_1_link" reason="Never"/>
+    <disable_collisions link1="right_robotiq_85_base_link" link2="right_wrist_2_link" reason="Never"/>
+    <disable_collisions link1="right_robotiq_85_base_link" link2="right_wrist_3_link" reason="Adjacent"/>
 </robot>

File: src/ur5e_gripper_moveit_config/urdf/ur5e_gripper.urdf.xacro (robot description, xacro)
@@ -4,9 +4,11 @@
     <link name="world"/>
     <xacro:include filename="single_ur5e_gripper.urdf.xacro" />
+    <!-- 左臂距离调整，需要根据桌子尺寸调整，不能被物理约束，否则会无法移动 -->
     <xacro:ur5e_gripper name="left_ur" prefix="" parent="world" initial_positions_file="$(arg initial_positions_file)">
-        <origin xyz="-0.275 0 1.03" rpy="0 0 0" />
+        <origin xyz="-0.65 0 1.016" rpy="0 0 0" />
     </xacro:ur5e_gripper>
+    <!-- 右臂距离调整 -->
     <xacro:ur5e_gripper name="right_ur" prefix="right_" parent="world" initial_positions_file="$(arg initial_positions_file)">
-        <origin xyz="1.075 0 1.03" rpy="0 0 3.1415926" />
+        <origin xyz="0.65 0 1.016" rpy="0 0 3.1415926" />
     </xacro:ur5e_gripper>
     <xacro:arg name="use_nominal_extrinsics" default="true"/>

Commit message: Dual Robotic Arm Grasp Collision Detection v1.0

File: src/ur5e_gripper_moveit_config/srdf/ur5e_gripper.srdf.xacro (robot description, xacro)
@@ -14,5 +14,5 @@
         <joint name="elbow_joint" value="1.5707" />
         <joint name="shoulder_lift_joint" value="-1.5707" />
-        <joint name="shoulder_pan_joint" value="0" />
+        <joint name="shoulder_pan_joint" value="0.7854" />
         <joint name="wrist_1_joint" value="-1.5707" />
         <joint name="wrist_2_joint" value="-1.5707" />
@@ -22,5 +22,13 @@
         <joint name="right_elbow_joint" value="1.5707" />
         <joint name="right_shoulder_lift_joint" value="-1.5707" />
-        <joint name="right_shoulder_pan_joint" value="0" />
+        <joint name="right_shoulder_pan_joint" value="-0.7854" />
+        <joint name="right_wrist_1_joint" value="-1.5707" />
+        <joint name="right_wrist_2_joint" value="-1.5707" />
+        <joint name="right_wrist_3_joint" value="0" />
+    </group_state>
+    <group_state name="right_local_wait" group="right_ur_manipulator">
+        <joint name="right_elbow_joint" value="1.5707" />
+        <joint name="right_shoulder_lift_joint" value="-1.5707" />
+        <joint name="right_shoulder_pan_joint" value="-1.0472" />
         <joint name="right_wrist_1_joint" value="-1.5707" />
         <joint name="right_wrist_2_joint" value="-1.5707" />
@@ -30,5 +38,5 @@
         <joint name="elbow_joint" value="1.5707" />
         <joint name="shoulder_lift_joint" value="-1.5707" />
-        <joint name="shoulder_pan_joint" value="0" />
+        <joint name="shoulder_pan_joint" value="0.7854" />
         <joint name="wrist_1_joint" value="-1.5707" />
         <joint name="wrist_2_joint" value="-1.5707" />
@@ -36,5 +44,5 @@
         <joint name="right_elbow_joint" value="1.5707" />
         <joint name="right_shoulder_lift_joint" value="-1.5707" />
-        <joint name="right_shoulder_pan_joint" value="0" />
+        <joint name="right_shoulder_pan_joint" value="-0.7854" />
         <joint name="right_wrist_1_joint" value="-1.5707" />
         <joint name="right_wrist_2_joint" value="-1.5707" />
